Commit message: fix(urdf): rename misleading 'lidar_3d' to 'tilted_lidar' + correct tilt axis
The sensor is a single-plane 2D LaserScan, not a 3D LiDAR. The previous
'lidar_3d' naming (suggested for disambiguation) was misleading.

Also fixes the tilt axis: rpy='-0.1 0 0' applied a ROLL (sideways
sweep) instead of a PITCH (forward/downward sweep). For detecting low
obstacles in front of the robot, the intended axis is pitch.

Changes:
- URDF link:  lidar_3d_link -> tilted_lidar_link
- URDF joint: rpy='-0.1 0 0' -> rpy='0 -0.1 0'
- Sensor name: laser_3d -> tilted_laser
- Topic: /scan_3d -> /scan_tilted
- nav2_params.yaml: update voxel_layer observation source
- nav2.launch.py: update info log message

File: src/navibot_description/urdf/navibot.urdf.xacro (robot description, xacro)
@@ -97,24 +97,27 @@
     <origin xyz="0 0 0" rpy="-${pi/2} 0 -${pi/2}"/>
   </joint>
-  <!-- ⭐ NOUVEAU : 3. LIDAR 3D ANTICOLISION (Rehaussé, inclinaison légère) ⭐ -->
-<link name="lidar_3d_link">
-  <visual>
-    <geometry><cylinder radius="0.04" length="0.05"/></geometry>
-    <material name="red"/>
-  </visual>
-  <collision>
-    <geometry><cylinder radius="0.04" length="0.05"/></geometry>
-  </collision>
-  <inertial>
-    <mass value="0.1"/>
-    <inertia ixx="0.0001" ixy="0" ixz="0" iyy="0.0001" iyz="0" izz="0.0001"/>
-  </inertial>
-</link>
-<joint name="lidar_3d_joint" type="fixed">
-  <parent link="base_link"/>
-  <child link="lidar_3d_link"/>
-  <!-- Position: avant du robot, centré, hauteur 0.2 m, inclinaison -0.1 rad (≈ -5.7°) -->
-  <origin xyz="${base_length/2 + 0.05} 0 0.2" rpy="-0.1 0 0"/>
-</joint>
+  <!-- 3. LIDAR 2D INCLINÉ — Anti-collision pour obstacles bas en avant -->
+  <!-- NB: ce capteur est un LaserScan 2D (un seul plan), pas un LiDAR 3D. -->
+  <link name="tilted_lidar_link">
+    <visual>
+      <geometry><cylinder radius="0.04" length="0.05"/></geometry>
+      <material name="red"/>
+    </visual>
+    <collision>
+      <geometry><cylinder radius="0.04" length="0.05"/></geometry>
+    </collision>
+    <inertial>
+      <mass value="0.1"/>
+      <inertia ixx="0.0001" ixy="0" ixz="0" iyy="0.0001" iyz="0" izz="0.0001"/>
+    </inertial>
+  </link>
+  <joint name="tilted_lidar_joint" type="fixed">
+    <parent link="base_link"/>
+    <child link="tilted_lidar_link"/>
+    <!-- Position: avant du robot, centré, hauteur 0.2 m.
+         Inclinaison: PITCH de -0.1 rad (≈ -5.7°) pour pointer vers le sol
+         devant le robot (axe Y = pitch, PAS roll). -->
+    <origin xyz="${base_length/2 + 0.05} 0 0.2" rpy="0 -0.1 0"/>
+  </joint>
   <!-- 4. IMU -->
   <link name="imu_link">
@@ -205,7 +208,7 @@
     </sensor>
   </gazebo>
-  <!-- ⭐ LiDAR 3D Anticollision Plugin (Demi-cercule vers le bas) ⭐ -->
-  <gazebo reference="lidar_3d_link">
-    <sensor type="ray" name="laser_3d">
+  <!-- LiDAR 2D INCLINÉ — demi-cercle avant pour anticollision basse -->
+  <gazebo reference="tilted_lidar_link">
+    <sensor type="ray" name="tilted_laser">
       <pose>0 0 0 0 0 0</pose>
       <visualize>true</visualize>
@@ -231,10 +234,10 @@
         </noise>
       </ray>
-      <plugin name="scan_plugin_3d" filename="libgazebo_ros_ray_sensor.so">
-        <ros>
-          <remapping>~/out:=/scan_3d</remapping>
+      <plugin name="tilted_scan_plugin" filename="libgazebo_ros_ray_sensor.so">
+        <ros>
+          <remapping>~/out:=/scan_tilted</remapping>
         </ros>
         <output_type>sensor_msgs/LaserScan</output_type>
-        <frame_name>lidar_3d_link</frame_name>
+        <frame_name>tilted_lidar_link</frame_name>
       </plugin>
     </sensor>

Commit message: rename: tilted_lidar -> lidar_obstacles_bas (noms en français)
Préférence du propriétaire du projet: cohérence linguistique avec le
reste du code (commentaires en français).

Renommage:
- link/joint: tilted_lidar_* -> lidar_obstacles_bas_*
- sensor:     tilted_laser   -> laser_obstacles_bas
- plugin:     tilted_scan_plugin -> plugin_scan_obstacles_bas
- topic:      /scan_tilted   -> /scan_obstacles_bas
- nav2_params.yaml et nav2.launch.py mis à jour en conséquence.

File: src/navibot_description/urdf/navibot.urdf.xacro (robot description, xacro)
@@ -99,5 +99,5 @@
   <!-- 3. LIDAR 2D INCLINÉ — Anti-collision pour obstacles bas en avant -->
   <!-- NB: ce capteur est un LaserScan 2D (un seul plan), pas un LiDAR 3D. -->
-  <link name="tilted_lidar_link">
+  <link name="lidar_obstacles_bas_link">
     <visual>
       <geometry><cylinder radius="0.04" length="0.05"/></geometry>
@@ -112,7 +112,7 @@
     </inertial>
   </link>
-  <joint name="tilted_lidar_joint" type="fixed">
+  <joint name="lidar_obstacles_bas_joint" type="fixed">
     <parent link="base_link"/>
-    <child link="tilted_lidar_link"/>
+    <child link="lidar_obstacles_bas_link"/>
     <!-- Position: avant du robot, centré, hauteur 0.2 m.
          Inclinaison: PITCH de -0.1 rad (≈ -5.7°) pour pointer vers le sol
@@ -209,6 +209,6 @@
   </gazebo>
   <!-- LiDAR 2D INCLINÉ — demi-cercle avant pour anticollision basse -->
-  <gazebo reference="tilted_lidar_link">
-    <sensor type="ray" name="tilted_laser">
+  <gazebo reference="lidar_obstacles_bas_link">
+    <sensor type="ray" name="laser_obstacles_bas">
       <pose>0 0 0 0 0 0</pose>
       <visualize>true</visualize>
@@ -234,10 +234,10 @@
         </noise>
       </ray>
-      <plugin name="tilted_scan_plugin" filename="libgazebo_ros_ray_sensor.so">
-        <ros>
-          <remapping>~/out:=/scan_tilted</remapping>
+      <plugin name="plugin_scan_obstacles_bas" filename="libgazebo_ros_ray_sensor.so">
+        <ros>
+          <remapping>~/out:=/scan_obstacles_bas</remapping>
         </ros>
         <output_type>sensor_msgs/LaserScan</output_type>
-        <frame_name>tilted_lidar_link</frame_name>
+        <frame_name>lidar_obstacles_bas_link</frame_name>
       </plugin>
     </sensor>

Commit message: tune(lidar_obstacles_bas): augmenter pitch de -0.1 à -0.2 rad
A -0.1 rad les rayons restaient presque horizontaux (constaté visuellement
dans RViz/Gazebo). A -0.2 rad le capteur descend assez pour détecter:
  - obstacles >= 10 cm à 2 m devant
  - obstacles >= 30 cm à 1 m devant

Le sol serait touché à 0.5/tan(0.2) ~ 2.46 m, ce qui dépasse la portée
max du capteur (2.0 m), donc pas de faux positif sur le sol.

File: src/navibot_description/urdf/navibot.urdf.xacro (robot description, xacro)
@@ -116,7 +116,11 @@
     <child link="lidar_obstacles_bas_link"/>
     <!-- Position: avant du robot, centré, hauteur 0.2 m.
-         Inclinaison: PITCH de -0.1 rad (≈ -5.7°) pour pointer vers le sol
-         devant le robot (axe Y = pitch, PAS roll). -->
-    <origin xyz="${base_length/2 + 0.05} 0 0.2" rpy="0 -0.1 0"/>
+         Inclinaison: PITCH de -0.2 rad (≈ -11.5°) pour pointer vers le sol
+         devant le robot (axe Y = pitch, PAS roll).
+         Géométrie: capteur à ~0.5 m du sol, portée max 2.0 m.
+         Le sol serait touché à d = 0.5/tan(0.2) ≈ 2.46 m, donc HORS portée:
+         pas de faux positifs sur le sol.
+         Détection garantie d'obstacles >= 10 cm à 2 m devant, >= 30 cm à 1 m. -->
+    <origin xyz="${base_length/2 + 0.05} 0 0.2" rpy="0 -0.2 0"/>
   </joint>
   <!-- 4. IMU -->

Commit message: fix(lidar_obstacles_bas): inverser le signe du pitch (-0.2 -> +0.2)
Constaté par l'utilisateur: avec rpy='0 -0.2 0' le capteur penche vers
le HAUT au lieu du bas.

Convention ROS REP-103: rotation autour de Y suit la règle de la main
droite. R_y(theta) appliqué à +X donne (cos theta, 0, -sin theta).
Donc theta POSITIF -> Z negatif -> avant qui penche VERS LE BAS.

J'avais inversé le signe dans l'analyse initiale. Le rendu visuel
d'Ismail (rayons partant vers le haut) confirme que +0.2 est la bonne
valeur pour pointer vers le sol.

File: src/navibot_description/urdf/navibot.urdf.xacro (robot description, xacro)
@@ -116,11 +116,13 @@
     <child link="lidar_obstacles_bas_link"/>
     <!-- Position: avant du robot, centré, hauteur 0.2 m.
-         Inclinaison: PITCH de -0.2 rad (≈ -11.5°) pour pointer vers le sol
+         Inclinaison: PITCH de +0.2 rad (≈ +11.5°) pour pointer vers le sol
          devant le robot (axe Y = pitch, PAS roll).
+         Convention ROS: R_y(+θ) bascule l'axe +X (avant) vers -Z (bas),
+         donc un pitch POSITIF fait pencher l'avant du capteur VERS LE BAS.
          Géométrie: capteur à ~0.5 m du sol, portée max 2.0 m.
          Le sol serait touché à d = 0.5/tan(0.2) ≈ 2.46 m, donc HORS portée:
          pas de faux positifs sur le sol.
          Détection garantie d'obstacles >= 10 cm à 2 m devant, >= 30 cm à 1 m. -->
-    <origin xyz="${base_length/2 + 0.05} 0 0.2" rpy="0 -0.2 0"/>
+    <origin xyz="${base_length/2 + 0.05} 0 0.2" rpy="0 0.2 0"/>
   </joint>
   <!-- IMPORTANT: empêcher Gazebo de "lumper" ce joint fixe dans base_link,

Commit message: improve(urdf): inertias correctes via xacro macros (box/cylinder)
Remplace les valeurs d'inertie 'à la main' (souvent fausses d'un facteur
2 à 9, comme ixx=iyy=0.01 sur une roue où la valeur correcte est 0.0056)
par des macros calculant les formules standard:
  - Boîte: I = (1/12)m·(...)
  - Cylindre: Ixx=Iyy=(1/12)m·(3r²+l²), Izz=(1/2)m·r²

Bénéfices:
- Inertias cohérentes avec la masse et la géométrie déclarée.
- Modifier une dimension (ex: wheel_radius) met à jour l'inertie auto.
- Plus de copier-coller fragile entre les 4 roues.

Aucun changement de masse ni de géométrie, donc le comportement dynamique
reste très proche; la simulation devient juste physiquement cohérente,
ce qui aide notamment Gazebo à intégrer la dynamique sans instabilités.

File: src/navibot_description/urdf/navibot.urdf.xacro (robot description, xacro)
@@ -15,4 +15,28 @@
   <material name="black"><color rgba="0.1 0.1 0.1 1.0"/></material>
   <material name="red"><color rgba="1.0 0.0 0.0 1.0"/></material>
+  <!-- ==================== MACROS D'INERTIE ==================== -->
+  <!-- Formules standard pour solides homogènes (référence: tout cours de
+       mécanique du solide). Évite les valeurs "à la main" qui peuvent
+       déstabiliser la simulation Gazebo si elles sont trop grossières. -->
+  <!-- Boîte alignée sur les axes du link (x=length, y=width, z=height) -->
+  <xacro:macro name="box_inertia" params="mass x y z">
+    <inertial>
+      <mass value="${mass}"/>
+      <inertia
+        ixx="${(1.0/12.0) * mass * (y*y + z*z)}" ixy="0" ixz="0"
+        iyy="${(1.0/12.0) * mass * (x*x + z*z)}" iyz="0"
+        izz="${(1.0/12.0) * mass * (x*x + y*y)}"/>
+    </inertial>
+  </xacro:macro>
+  <!-- Cylindre dont l'axe coïncide avec Z du link -->
+  <xacro:macro name="cylinder_inertia" params="mass radius length">
+    <inertial>
+      <mass value="${mass}"/>
+      <inertia
+        ixx="${(1.0/12.0) * mass * (3.0*radius*radius + length*length)}" ixy="0" ixz="0"
+        iyy="${(1.0/12.0) * mass * (3.0*radius*radius + length*length)}" iyz="0"
+        izz="${0.5 * mass * radius*radius}"/>
+    </inertial>
+  </xacro:macro>
   <!-- BASE_LINK -->
   <link name="base_footprint"/>
@@ -24,5 +48,5 @@
     <visual><geometry><box size="${base_length} ${base_width} ${base_height}"/></geometry><material name="blue"/></visual>
     <collision><geometry><box size="${base_length} ${base_width} ${base_height}"/></geometry></collision>
-    <inertial><mass value="40.0"/><inertia ixx="2.0" ixy="0" ixz="0" iyy="3.0" iyz="0" izz="4.0"/></inertial>
+    <xacro:box_inertia mass="40.0" x="${base_length}" y="${base_width}" z="${base_height}"/>
   </link>
    <!-- ==================== ROUES (MACRO AVEC LIMITES) ==================== -->
@@ -31,5 +55,5 @@
       <visual><geometry><cylinder radius="${wheel_radius}" length="${wheel_width}"/></geometry><material name="black"/></visual>
       <collision><geometry><cylinder radius="${wheel_radius}" length="${wheel_width}"/></geometry></collision>
-      <inertial><mass value="2.0"/><inertia ixx="0.01" ixy="0" ixz="0" iyy="0.01" iyz="0" izz="0.01"/></inertial>
+      <xacro:cylinder_inertia mass="2.0" radius="${wheel_radius}" length="${wheel_width}"/>
     </link>
     <joint name="${prefix}_wheel_joint" type="continuous">
@@ -48,5 +72,5 @@
     <visual><geometry><cylinder radius="${wheel_radius}" length="${wheel_width}"/></geometry><material name="black"/></visual>
     <collision><geometry><cylinder radius="${wheel_radius}" length="${wheel_width}"/></geometry></collision>
-    <inertial><mass value="2"/><inertia ixx="0.01" ixy="0" ixz="0" iyy="0.01" iyz="0" izz="0.01"/></inertial>
+    <xacro:cylinder_inertia mass="2.0" radius="${wheel_radius}" length="${wheel_width}"/>
   </link>
   <joint name="rear_left_wheel_joint" type="continuous">
@@ -60,5 +84,5 @@
     <visual><geometry><cylinder radius="${wheel_radius}" length="${wheel_width}"/></geometry><material name="black"/></visual>
     <collision><geometry><cylinder radius="${wheel_radius}" length="${wheel_width}"/></geometry></collision>
-    <inertial><mass value="2"/><inertia ixx="0.01" ixy="0" ixz="0" iyy="0.01" iyz="0" izz="0.01"/></inertial>
+    <xacro:cylinder_inertia mass="2.0" radius="${wheel_radius}" length="${wheel_width}"/>
   </link>
   <joint name="rear_right_wheel_joint" type="continuous">
@@ -74,5 +98,5 @@
     <visual><geometry><cylinder radius="0.06" length="0.08"/></geometry><material name="red"/></visual>
     <collision><geometry><cylinder radius="0.06" length="0.08"/></geometry></collision>
-    <inertial><mass value="0.5"/><inertia ixx="0.0001" ixy="0" ixz="0" iyy="0.0001" iyz="0" izz="0.0001"/></inertial>
+    <xacro:cylinder_inertia mass="0.5" radius="0.06" length="0.08"/>
   </link>
   <joint name="lidar_joint" type="fixed">
@@ -85,5 +109,5 @@
     <visual><geometry><box size="0.05 0.08 0.03"/></geometry></visual>
     <collision><geometry><box size="0.05 0.08 0.03"/></geometry></collision>
-    <inertial><mass value="0.1"/><inertia ixx="0.0001" ixy="0" ixz="0" iyy="0.0001" iyz="0" izz="0.0001"/></inertial>
+    <xacro:box_inertia mass="0.1" x="0.05" y="0.08" z="0.03"/>
   </link>
   <joint name="camera_joint" type="fixed">
@@ -107,8 +131,5 @@
       <geometry><cylinder radius="0.04" length="0.05"/></geometry>
     </collision>
-    <inertial>
-      <mass value="0.1"/>
-      <inertia ixx="0.0001" ixy="0" ixz="0" iyy="0.0001" iyz="0" izz="0.0001"/>
-    </inertial>
+    <xacro:cylinder_inertia mass="0.1" radius="0.04" length="0.05"/>
   </link>
   <joint name="lidar_obstacles_bas_joint" type="fixed">
@@ -136,5 +157,5 @@
   <link name="imu_link">
     <visual><geometry><box size="0.02 0.02 0.01"/></geometry></visual>
-    <inertial><mass value="0.01"/><inertia ixx="0.00001" ixy="0" ixz="0" iyy="0.00001" iyz="0" izz="0.00001"/></inertial>
+    <xacro:box_inertia mass="0.01" x="0.02" y="0.02" z="0.01"/>
   </link>
   <joint name="imu_joint" type="fixed">
